Commit message: Muchas mejoras y traslados de ciertas simulaciones

File: quadruped_description/urdf/quadruped_robot.xacro (robot description, xacro)
@@ -1,8 +1,6 @@
-<robot name="quadruped" >
+<?xml version="1.0"?>
+<robot xmlns:xacro="http://www.ros.org/wiki/xacro">
   <link name="dummy">
   </link>
-  <material name="black">
-    <color rgba="0 0 0 0.5"/>
-  </material>
   <joint name="dummy_joint" type="fixed">
      <parent link="dummy"/>
@@ -21,5 +19,5 @@
         <mesh filename="package://quadruped_description/meshes/frame_aluminum_motor_case.stl"/>
       </geometry>
-      <material name="black"/>
+      <material name="grey"/>
     </visual>
     <collision>
@@ -45,5 +43,5 @@
         <mesh filename="package://quadruped_description/meshes/joint_gear_upper_assembly.stl"/>
       </geometry>
-      <material name="black"/>
+      <material name="grey"/>
     </visual>
     <collision>
@@ -69,5 +67,5 @@
         <mesh filename="package://quadruped_description/meshes/joint_gear_upper_assembly.stl"/>
       </geometry>
-      <material name="black"/>
+      <material name="grey"/>
     </visual>
     <collision>
@@ -93,5 +91,5 @@
         <mesh filename="package://quadruped_description/meshes/joint_gear_upper_assembly.stl"/>
       </geometry>
-      <material name="black"/>
+      <material name="grey"/>
     </visual>
     <collision>
@@ -117,5 +115,5 @@
         <mesh filename="package://quadruped_description/meshes/joint_gear_upper_assembly.stl"/>
       </geometry>
-      <material name="black"/>
+      <material name="grey"/>
     </visual>
     <collision>
@@ -141,5 +139,5 @@
         <mesh filename="package://quadruped_description/meshes/Assembly_lower_link_v2.stl"/>
       </geometry>
-      <material name="black"/>
+      <material name="grey"/>
     </visual>
     <collision>
@@ -165,5 +163,5 @@
         <mesh filename="package://quadruped_description/meshes/Assembly_lower_link_v2.stl"/>
       </geometry>
-      <material name="black"/>
+      <material name="grey"/>
     </visual>
     <collision>
@@ -189,5 +187,5 @@
         <mesh filename="package://quadruped_description/meshes/Assembly_lower_link_v2.stl"/>
       </geometry>
-      <material name="black"/>
+      <material name="grey"/>
     </visual>
     <collision>
@@ -213,5 +211,5 @@
         <mesh filename="package://quadruped_description/meshes/Assembly_lower_link_v2.stl"/>
       </geometry>
-      <material name="black"/>
+      <material name="grey"/>
     </visual>
     <collision>

Commit message: SE spawneo el robot en gazebo

File: quadruped_description/urdf/quadruped_robot.xacro (robot description, xacro)
@@ -3,8 +3,4 @@
   <link name="dummy">
   </link>
-  <joint name="dummy_joint" type="fixed">
-     <parent link="dummy"/>
-     <child link="body"/>
-  </joint>
   <link name="body">
     <inertial>
@@ -17,18 +13,21 @@
       <origin rpy="1.57 0 1.57" xyz="0 0 0"/>
       <geometry>
-        <mesh filename="package://quadruped_description/meshes/frame_aluminum_motor_case.stl"/>
-      </geometry>
-      <material name="grey"/>
-    </visual>
-    <collision>
-      <origin
-        xyz="0 0 0"
-        rpy="1.57 0 1.57" />
-      <geometry>
-        <mesh
-          filename="package://quadruped_description/meshes/frame_aluminum_motor_case.stl" />
-      </geometry>
-    </collision>
-  </link>
+        <mesh filename="model://my_quadruped/meshes/frame_aluminum_motor_case.dae" />
+      </geometry>
+      <material name="grey"/>
+    </visual>
+    <collision>
+      <origin
+        xyz="0 0 0"
+        rpy="1.57 0 1.57" />
+      <geometry>
+        <mesh filename="model://my_quadruped/meshes/frame_aluminum_motor_case.dae" />
+      </geometry>
+    </collision>
+  </link>
+  <joint name="dummy_joint" type="fixed">
+     <parent link="dummy"/>
+     <child link="body"/>
+  </joint>
   <link name="front_left_u">
     <inertial>
@@ -41,15 +40,14 @@
       <origin rpy="1.57 0 1.57" xyz="0 0 0"/>
       <geometry>
-        <mesh filename="package://quadruped_description/meshes/joint_gear_upper_assembly.stl"/>
-      </geometry>
-      <material name="grey"/>
-    </visual>
-    <collision>
-      <origin
-        xyz="0 0 0"
-        rpy="1.57 0 1.57" />
-      <geometry>
-        <mesh
-          filename="package://quadruped_description/meshes/joint_gear_upper_assembly.stl" />
+        <mesh filename="model://my_quadruped/meshes/joint_gear_upper_assembly.stl" />
+      </geometry>
+      <material name="grey"/>
+    </visual>
+    <collision>
+      <origin
+        xyz="0 0 0"
+        rpy="1.57 0 1.57" />
+      <geometry>
+        <mesh filename="model://my_quadruped/meshes/joint_gear_upper_assembly.stl" />
       </geometry>
     </collision>
@@ -65,5 +63,5 @@
       <origin rpy="1.57 3.14 1.57" xyz="0 0 0"/>
       <geometry>
-        <mesh filename="package://quadruped_description/meshes/joint_gear_upper_assembly.stl"/>
+        <mesh filename="model://my_quadruped/meshes/joint_gear_upper_assembly.stl" />
       </geometry>
       <material name="grey"/>
@@ -74,6 +72,5 @@
         rpy="1.57 3.14 1.57" />
       <geometry>
-        <mesh
-          filename="package://quadruped_description/meshes/joint_gear_upper_assembly.stl" />
+        <mesh filename="model://my_quadruped/meshes/joint_gear_upper_assembly.stl" />
       </geometry>
     </collision>
@@ -89,5 +86,5 @@
       <origin rpy="1.57 3.14 1.57" xyz="0 0 0"/>
       <geometry>
-        <mesh filename="package://quadruped_description/meshes/joint_gear_upper_assembly.stl"/>
+        <mesh filename="model://my_quadruped/meshes/joint_gear_upper_assembly.stl" />
       </geometry>
       <material name="grey"/>
@@ -98,6 +95,5 @@
         rpy="1.57 3.14 1.57" />
       <geometry>
-        <mesh
-          filename="package://quadruped_description/meshes/joint_gear_upper_assembly.stl" />
+        <mesh filename="model://my_quadruped/meshes/joint_gear_upper_assembly.stl" />
       </geometry>
     </collision>
@@ -113,15 +109,14 @@
       <origin rpy="1.57 0 1.57" xyz="0 0 0"/>
       <geometry>
-        <mesh filename="package://quadruped_description/meshes/joint_gear_upper_assembly.stl"/>
-      </geometry>
-      <material name="grey"/>
-    </visual>
-    <collision>
-      <origin
-        xyz="0 0 0"
-        rpy="1.57 0 1.57" />
-      <geometry>
-        <mesh
-          filename="package://quadruped_description/meshes/joint_gear_upper_assembly.stl" />
+        <mesh filename="model://my_quadruped/meshes/joint_gear_upper_assembly.stl" />
+      </geometry>
+      <material name="grey"/>
+    </visual>
+    <collision>
+      <origin
+        xyz="0 0 0"
+        rpy="1.57 0 1.57" />
+      <geometry>
+        <mesh filename="model://my_quadruped/meshes/joint_gear_upper_assembly.stl" />
       </geometry>
     </collision>
@@ -137,15 +132,14 @@
       <origin rpy="1.57 0 1.57" xyz="0 0 0"/>
       <geometry>
-        <mesh filename="package://quadruped_description/meshes/Assembly_lower_link_v2.stl"/>
-      </geometry>
-      <material name="grey"/>
-    </visual>
-    <collision>
-      <origin
-        xyz="0 0 0"
-        rpy="1.57 0 1.57" />
-      <geometry>
-        <mesh
-          filename="package://quadruped_description/meshes/Assembly_lower_link_v2.stl" />
+        <mesh filename="model://my_quadruped/meshes/Assembly_lower_link_v2.stl" />
+      </geometry>
+      <material name="grey"/>
+    </visual>
+    <collision>
+      <origin
+        xyz="0 0 0"
+        rpy="1.57 0 1.57" />
+      <geometry>
+        <mesh filename="model://my_quadruped/meshes/Assembly_lower_link_v2.stl" />
       </geometry>
     </collision>
@@ -161,5 +155,5 @@
       <origin rpy="-1.57 0 -1.57" xyz="0 0 0"/>
       <geometry>
-        <mesh filename="package://quadruped_description/meshes/Assembly_lower_link_v2.stl"/>
+        <mesh filename="model://my_quadruped/meshes/Assembly_lower_link_v2.stl" />
       </geometry>
       <material name="grey"/>
@@ -170,6 +164,5 @@
         rpy="-1.57 0 -1.57" />
       <geometry>
-        <mesh
-          filename="package://quadruped_description/meshes/Assembly_lower_link_v2.stl" />
+        <mesh filename="model://my_quadruped/meshes/Assembly_lower_link_v2.stl" />
       </geometry>
     </collision>
@@ -185,5 +178,5 @@
       <origin rpy="-1.57 0 -1.57" xyz="0 0 0"/>
       <geometry>
-        <mesh filename="package://quadruped_description/meshes/Assembly_lower_link_v2.stl"/>
+        <mesh filename="model://my_quadruped/meshes/Assembly_lower_link_v2.stl" />
       </geometry>
       <material name="grey"/>
@@ -194,6 +187,5 @@
         rpy="-1.57 0 -1.57" />
       <geometry>
-        <mesh
-          filename="package://quadruped_description/meshes/Assembly_lower_link_v2.stl" />
+        <mesh filename="model://my_quadruped/meshes/Assembly_lower_link_v2.stl" />
       </geometry>
     </collision>
@@ -209,15 +201,14 @@
       <origin rpy="1.57 0 1.57" xyz="0 0 0"/>
       <geometry>
-        <mesh filename="package://quadruped_description/meshes/Assembly_lower_link_v2.stl"/>
-      </geometry>
-      <material name="grey"/>
-    </visual>
-    <collision>
-      <origin
-        xyz="0 0 0"
-        rpy="1.57 0 1.57" />
-      <geometry>
-        <mesh
-          filename="package://quadruped_description/meshes/Assembly_lower_link_v2.stl" />
+        <mesh filename="model://my_quadruped/meshes/Assembly_lower_link_v2.stl" />
+      </geometry>
+      <material name="grey"/>
+    </visual>
+    <collision>
+      <origin
+        xyz="0 0 0"
+        rpy="1.57 0 1.57" />
+      <geometry>
+        <mesh filename="model://my_quadruped/meshes/Assembly_lower_link_v2.stl" />
       </geometry>
     </collision>
