Commit message: Se incorpora el urdf modificado y los arreglos en gazebo para el nuevo joint de la camara

File: quadruped_description/urdf/quadruped.urdf (robot description, URDF)
Before this commit: robot quadruped, 10 links, 9 joints
Links:
- added link camera_link, mass 0.046222; collision mesh filename=package://quadruped_description/meshes/camera_link.stl; visual mesh filename=package://quadruped_description/meshes/camera_link.stl
- link body: mass 8.4 -> 3.0416
Joints:
- added joint camera_joint: type revolute, parent body, child camera_link, origin xyz=0.2 0 0.42525 rpy=0 0 0, axis 0 1 0, limit lower=-3.14 upper=3.14 effort=100 velocity=100

File: quadruped_description/urdf/quadruped_robot.xacro (robot description, xacro)
@@ -5,22 +5,27 @@
   <link name="body">
     <inertial>
-      <mass value="8.4" />
-      <inertia ixx="0.14596" ixy="0.00010"  ixz="0.00013"
-               iyy="0.08855" iyz="-0.03467"
-               izz="0.11796" />
-    </inertial>
-    <visual>
-      <origin rpy="1.57 0 1.57" xyz="0 0 0"/>
-      <geometry>
-        <mesh filename="model://my_quadruped/meshes/frame_aluminum_motor_case.dae" />
-      </geometry>
-      <material name="grey"/>
-    </visual>
-    <collision>
-      <origin
-        xyz="0 0 0"
-        rpy="1.57 0 1.57" />
-      <geometry>
-        <mesh filename="model://my_quadruped/meshes/frame_aluminum_motor_case.dae" />
+      <mass
+        value="3.0416" />
+      <inertia
+        ixx="0.0073301"
+        ixy="2.1671E-09"
+        ixz="1.9602E-06"
+        iyy="0.0077176"
+        iyz="-1.1292E-05"
+        izz="0.0059691" />
+    </inertial>
+    <visual>
+      <origin rpy="0 0 ${pi / 2.0}" xyz="0 0 -0.06"/>
+      <geometry>
+        <mesh filename="model://my_quadruped/meshes/frame_aluminum_motor.stl" />
+      </geometry>
+      <material name="grey"/>
+    </visual>
+    <collision>
+      <origin
+        xyz="0 0 -0.06"
+        rpy="0 0 ${pi / 2.0}" />
+      <geometry>
+        <mesh filename="model://my_quadruped/meshes/frame_aluminum_motor.stl" />
       </geometry>
     </collision>
@@ -29,4 +34,58 @@
      <parent link="dummy"/>
      <child link="body"/>
+  </joint>
+  <link
+    name="camera_link">
+    <inertial>
+      <mass
+        value="0.046222" />
+      <inertia
+        ixx="2.633E-06"
+        ixy="-4.2166E-09"
+        ixz="1.2531E-08"
+        iyy="2.5049E-05"
+        iyz="9.9718E-08"
+        izz="2.639E-05" />
+    </inertial>
+    <visual>
+      <origin
+        xyz="0 0 0"
+        rpy="${pi / 2.0} 0 ${pi / 2.0}" />
+      <geometry>
+        <mesh
+          filename="model://my_quadruped/meshes/camera_link.stl" />
+      </geometry>
+      <material
+        name="">
+        <color
+          rgba="0.75294 0.75294 0.75294 1" />
+      </material>
+    </visual>
+    <collision>
+      <origin
+        xyz="0 0 0"
+        rpy="0 0 0" />
+      <geometry>
+        <mesh
+          filename="model://my_quadruped/meshes/camera_link.stl" />
+      </geometry>
+    </collision>
+  </link>
+  <joint
+    name="camera_joint" type="revolute">
+    <origin
+      xyz="0.2 0 0.42525"
+      rpy="0 0 0" />
+    <parent
+      link="body" />
+    <child
+      link="camera_link" />
+    <axis
+      xyz="0 1 0" />
+    <limit
+      lower="-3.14"
+      upper="3.14"
+      effort="100"
+      velocity="100" />
   </joint>
   <link name="front_left_u">
@@ -53,4 +112,11 @@
     </collision>
   </link>
+  <joint name="front_left_joint1" type="revolute">
+    <limit effort="1000.0" lower="-3.14" upper="3.14" velocity="0.5"/>
+    <parent link="body"/>
+    <child link="front_left_u"/>
+    <origin xyz="0.11 0.05 0" rpy="0 0 0" />
+    <axis xyz="0 1 0" />
+  </joint>
   <link name="front_right_u">
     <inertial>
@@ -228,11 +294,4 @@
     <axis xyz="0 1 0" />
   </joint>
-  <joint name="front_left_joint1" type="revolute">
-    <limit effort="1000.0" lower="-3.14" upper="3.14" velocity="0.5"/>
-    <parent link="body"/>
-    <child link="front_left_u"/>
-    <origin xyz="0.11 0.05 0" rpy="0 0 0" />
-    <axis xyz="0 1 0" />
-  </joint>
   <joint name="front_left_joint2" type="revolute">
     <limit effort="1000.0" lower="-3.14" upper="3.14" velocity="0.5"/>
