Commit message: Se realizo la communicacion para coppellia y para gazebo

File: quadruped_description/urdf/quadruped.urdf.xacro (robot description, xacro)
@@ -3,5 +3,5 @@
     <!-- LLamado de los otros xacros -->
     <xacro:include filename="common_properties.urdf.xacro" />
-    <xacro:include filename="quadruped_robot.urdf.xacro" />
+    <xacro:include filename="quadruped_robot3.urdf.xacro" />
     <xacro:include filename="quadruped_gazebo.urdf.xacro" />
 </robot>

File: quadruped_description/urdf/quadruped_gazebo.urdf.xacro (robot description, xacro)
@@ -20,4 +20,20 @@
     <mu1>0.20</mu1>
     <mu2>0.20</mu2>
+  </gazebo>
+  <gazebo reference="front_left_d_contact_link">
+    <mu1>1.0</mu1>
+    <mu2>1.0</mu2>
+  </gazebo>
+  <gazebo reference="front_right_d_contact_link">
+    <mu1>1.0</mu1>
+    <mu2>1.0</mu2>
+  </gazebo>
+  <gazebo reference="back_left_d_contact_link">
+    <mu1>1.0</mu1>
+    <mu2>1.0</mu2>
+  </gazebo>
+  <gazebo reference="front_right_d_contact_link">
+    <mu1>1.0</mu1>
+    <mu2>1.0</mu2>
   </gazebo>
   <ros2_control name="GazeboSystem" type="system">

File: quadruped_description/urdf/quadruped_robot2.urdf.xacro (robot description, xacro)
@@ -7,5 +7,5 @@
       <origin rpy="0 ${pi /8} 0" xyz="0 0 0.05"/>
       <mass
-        value="15" />
+        value="5" />
       <!-- <inertia
         ixx="0.04" ixy="-0.000009" ixz="0.0045"
@@ -13,7 +13,7 @@
         izz="0.03" /> -->
       <inertia
-        ixx="0.08" ixy="-0.0000173" ixz="0.00929"
-        iyy="0.08613" iyz="-0.0000446"
-        izz="0.0601" />
+        ixx="0.04" ixy="-0.0000093" ixz="0.00429"
+        iyy="0.04613" iyz="-0.0000226"
+        izz="0.0301" />
     </inertial>
     <visual>
@@ -36,4 +36,5 @@
     name="camera_link">
     <inertial>
+      <origin rpy="0 0 0" xyz="0 0 0"/>
       <mass
         value="0.05" />
@@ -69,11 +70,9 @@
   <link name="front_left_u">
     <inertial>
-      <mass value="0.8" />
-      <!-- <inertia ixx="0.00025" ixy="0.0012"  ixz="0.0"
-               iyy="0.022" iyz="0.0"
-               izz="0.022" /> -->
-      <inertia ixx="0.00051" ixy="0.0025"  ixz="0.0"
-               iyy="0.044" iyz="0.0"
-               izz="0.044" />
+      <origin rpy="0 0 0.08" xyz="0.1 0 0"/>
+      <mass value="0.8" />
+      <inertia ixx="0.00006" ixy="0.0003"  ixz="0.0"
+               iyy="0.005" iyz="0.0"
+               izz="0.005" />
     </inertial>
     <visual>
@@ -95,11 +94,9 @@
   <link name="front_right_u">
     <inertial>
-      <mass value="0.8" />
-      <!-- <inertia ixx="0.00035" ixy="-0.0019"  ixz="0.0"
-               iyy="0.022" iyz="0.0"
-               izz="0.022" /> -->
-      <inertia ixx="0.00076" ixy="-0.00385"  ixz="0.0"
-               iyy="0.044" iyz="0.0"
-               izz="0.044" />
+      <origin rpy="0 0 -0.08" xyz="0.1 0 0"/>
+      <mass value="0.8" />
+      <inertia ixx="0.00006" ixy="-0.0003"  ixz="0.0"
+               iyy="0.005" iyz="0.0"
+               izz="0.005" />
     </inertial>
     <visual>
@@ -121,11 +118,9 @@
   <link name="back_left_u">
     <inertial>
-      <mass value="0.8" />
-      <!-- <inertia ixx="0.00035" ixy="-0.0019"  ixz="0.0"
-               iyy="0.022" iyz="0.0"
-               izz="0.022" /> -->
-      <inertia ixx="0.00076" ixy="-0.00385"  ixz="0.0"
-               iyy="0.044" iyz="0.0"
-               izz="0.044" />
+      <origin rpy="0 0 -0.08" xyz="0.1 0 0"/>
+      <mass value="0.8" />
+      <inertia ixx="0.00006" ixy="-0.0003"  ixz="0.0"
+               iyy="0.005" iyz="0.0"
+               izz="0.005" />
     </inertial>
     <visual>
@@ -147,11 +142,9 @@
   <link name="back_right_u">
     <inertial>
-      <mass value="0.8" />
-      <!-- <inertia ixx="0.00025" ixy="0.0012"  ixz="0.0"
-               iyy="0.022" iyz="0.0"
-               izz="0.022" /> -->
-      <inertia ixx="0.00051" ixy="0.0025"  ixz="0.0"
-               iyy="0.044" iyz="0.0"
-               izz="0.044" />
+      <origin rpy="0 0 0.08" xyz="0.1 0 0"/>
+      <mass value="0.8" />
+      <inertia ixx="0.00006" ixy="0.0003"  ixz="0.0"
+               iyy="0.005" iyz="0.0"
+               izz="0.005" />
     </inertial>
     <visual>
@@ -173,14 +166,9 @@
   <link name="front_left_d">
     <inertial>
-      <mass value="1.0" />
-      <!-- <inertia ixx="0.0039" ixy="0.012"  ixz="0.0"
-               iyy="0.1412" iyz="0.0"
-               izz="0.1447" /> Pata nueva-->
-      <!-- <inertia ixx="0.000045" ixy="0.0019"  ixz="0.0"
-               iyy="0.022" iyz="0.0"
-               izz="0.022" /> -->
-      <inertia ixx="0.0009" ixy="0.0038"  ixz="0.0"
-               iyy="0.044" iyz="0.0"
-               izz="0.0457" />
+      <origin rpy="0 0 0.08" xyz="0.15 0 0"/>
+      <mass value="0.8" />
+      <inertia ixx="0.00011" ixy="0.00045"  ixz="0.0"
+               iyy="0.006" iyz="0.0"
+               izz="0.006" />
     </inertial>
     <visual>
@@ -202,11 +190,9 @@
   <link name="front_right_d">
     <inertial>
-      <mass value="1.0" />
-      <!-- <inertia ixx="0.000045" ixy="-0.0019"  ixz="0.0"
-               iyy="0.022" iyz="0.0"
-               izz="0.022" /> -->
-      <inertia ixx="0.0009" ixy="-0.0038"  ixz="0.0"
-               iyy="0.044" iyz="0.0"
-               izz="0.0457" />
+      <origin rpy="0 0 -0.08" xyz="0.15 0 0"/>
+      <mass value="0.8" />
+      <inertia ixx="0.00011" ixy="-0.00045"  ixz="0.0"
+               iyy="0.006" iyz="0.0"
+               izz="0.006" />
     </inertial>
     <visual>
@@ -228,11 +214,9 @@
   <link name="back_left_d">
     <inertial>
-      <mass value="1.0" />
-      <!-- <inertia ixx="0.000045" ixy="-0.0019"  ixz="0.0"
-               iyy="0.022" iyz="0.0"
-               izz="0.022" /> -->
-      <inertia ixx="0.0009" ixy="-0.0038"  ixz="0.0"
-               iyy="0.044" iyz="0.0"
-               izz="0.0457" />
+      <origin rpy="0 0 -0.08" xyz="0.15 0 0"/>
+      <mass value="0.8" />
+      <inertia ixx="0.00011" ixy="-0.00045"  ixz="0.0"
+               iyy="0.006" iyz="0.0"
+               izz="0.006" />
     </inertial>
     <visual>
@@ -254,11 +238,9 @@
   <link name="back_right_d">
     <inertial>
-      <mass value="1.0" />
-      <!-- <inertia ixx="0.000045" ixy="0.0019"  ixz="0.0"
-               iyy="0.022" iyz="0.0"
-               izz="0.022" /> -->
-      <inertia ixx="0.0009" ixy="0.0038"  ixz="0.0"
-               iyy="0.044" iyz="0.0"
-               izz="0.0457" />
+      <origin rpy="0 0 0.08" xyz="0.15 0 0"/>
+      <mass value="0.8" />
+      <inertia ixx="0.00011" ixy="0.00045"  ixz="0.0"
+               iyy="0.006" iyz="0.0"
+               izz="0.006" />
     </inertial>
     <visual>
@@ -278,4 +260,112 @@
     </collision>
   </link>
+  <link name="front_left_d_contact_link">
+    <inertial>
+      <mass value="0.01" />
+      <origin xyz="0 0 0" />
+      <inertia ixx="1e-5" ixy="0" ixz="0" iyy="1e-5" iyz="0" izz="1e-5" />
+    </inertial>
+    <visual>
+      <origin xyz="0 0.05 0" rpy="${pi/2} 0 0" />
+      <geometry>
+        <cylinder radius="0.018" length="0.19" />
+      </geometry>
+      <material name="grey">
+        <color rgba="0.5 0.5 0.5 1" />
+      </material>
+    </visual>
+    <collision>
+      <origin xyz="0 0.05 0" rpy="${pi/2} 0 0" />
+      <geometry>
+        <cylinder radius="0.018" length="0.19" />
+      </geometry>
+    </collision>
+  </link>
+  <joint name="front_left_d_contact_joint" type="fixed">
+    <parent link="front_left_d" /> <!-- Nombre del link actual de la pata -->
+    <child link="front_left_d_contact_link" />
+    <origin xyz="0.4 0 0" rpy="0 0 0" /> <!-- Ajusta la posición al final de la pata -->
+  </joint>
+  <link name="front_right_d_contact_link">
+    <inertial>
+      <mass value="0.01" />
+      <origin xyz="0 0 0" />
+      <inertia ixx="1e-5" ixy="0" ixz="0" iyy="1e-5" iyz="0" izz="1e-5" />
+    </inertial>
+    <visual>
+      <origin xyz="0 -0.05 0" rpy="${pi/2} 0 0" />
+      <geometry>
+        <cylinder radius="0.018" length="0.19" />
+      </geometry>
+      <material name="grey">
+        <color rgba="0.5 0.5 0.5 1" />
+      </material>
+    </visual>
+    <collision>
+      <origin xyz="0 -0.05 0" rpy="${pi/2} 0 0" />
+      <geometry>
+        <cylinder radius="0.018" length="0.19" />
+      </geometry>
+    </collision>
+  </link>
+  <joint name="front_right_d_contact_joint" type="fixed">
+    <parent link="front_right_d" /> <!-- Nombre del link actual de la pata -->
+    <child link="front_right_d_contact_link" />
+    <origin xyz="0.4 0 0" rpy="0 0 0" /> <!-- Ajusta la posición al final de la pata -->
+  </joint>
+  <link name="back_right_d_contact_link">
+    <inertial>
+      <mass value="0.01" />
+      <origin xyz="0 0 0" />
+      <inertia ixx="1e-5" ixy="0" ixz="0" iyy="1e-5" iyz="0" izz="1e-5" />
+    </inertial>
+    <visual>
+      <origin xyz="0 0.05 0" rpy="${pi/2} 0 0" />
+      <geometry>
+        <cylinder radius="0.018" length="0.19" />
+      </geometry>
+      <material name="grey">
+        <color rgba="0.5 0.5 0.5 1" />
+      </material>
+    </visual>
+    <collision>
+      <origin xyz="0 0.05 0" rpy="${pi/2} 0 0" />
+      <geometry>
+        <cylinder radius="0.018" length="0.19" />
+      </geometry>
+    </collision>
+  </link>
+  <joint name="back_right_d_contact_joint" type="fixed">
+    <parent link="back_right_d" /> <!-- Nombre del link actual de la pata -->
+    <child link="back_right_d_contact_link" />
+    <origin xyz="0.4 0 0" rpy="0 0 0" /> <!-- Ajusta la posición al final de la pata -->
+  </joint>
+   <link name="back_left_d_contact_link">
+    <inertial>
+      <mass value="0.01" />
+      <origin xyz="0 0 0" />
+      <inertia ixx="1e-5" ixy="0" ixz="0" iyy="1e-5" iyz="0" izz="1e-5" />
+    </inertial>
+    <visual>
+      <origin xyz="0 -0.05 0" rpy="${pi/2} 0 0" />
+      <geometry>
+        <cylinder radius="0.018" length="0.19" />
+      </geometry>
+      <material name="grey">
+        <color rgba="0.5 0.5 0.5 1" />
+      </material>
+    </visual>
+    <collision>
+      <origin xyz="0 -0.05 0" rpy="${pi/2} 0 0" />
+      <geometry>
+        <cylinder radius="0.018" length="0.19" />
+      </geometry>
+    </collision>
+  </link>
+  <joint name="back_left_d_contact_joint" type="fixed">
+    <parent link="back_left_d" /> <!-- Nombre del link actual de la pata -->
+    <child link="back_left_d_contact_link" />
+    <origin xyz="0.4 0 0" rpy="0 0 0" /> <!-- Ajusta la posición al final de la pata -->
+  </joint>
   <joint name="dummy_joint" type="fixed">
      <parent link="dummy"/>
@@ -355,111 +445,3 @@
     <axis xyz="0 1 0" />
   </joint>
-  <link name="front_left_d_contact_link">
-    <inertial>
-      <mass value="0.01" />
-      <origin xyz="0 0 0" />
-      <inertia ixx="1e-5" ixy="0" ixz="0" iyy="1e-5" iyz="0" izz="1e-5" />
-    </inertial>
-    <visual>
-      <origin xyz="0 0.05 0" rpy="${pi/2} 0 0" />
-      <geometry>
-        <cylinder radius="0.018" length="0.19" />
-      </geometry>
-      <material name="grey">
-        <color rgba="0.5 0.5 0.5 1" />
-      </material>
-    </visual>
-    <collision>
-      <origin xyz="0 0.05 0" rpy="${pi/2} 0 0" />
-      <geometry>
-        <cylinder radius="0.018" length="0.19" />
-      </geometry>
-    </collision>
-  </link>
-  <joint name="front_left_d_contact_joint" type="fixed">
-    <parent link="front_left_d" /> <!-- Nombre del link actual de la pata -->
-    <child link="front_left_d_contact_link" />
-    <origin xyz="0.4 0 0" rpy="0 0 0" /> <!-- Ajusta la posición al final de la pata -->
-  </joint>
-  <link name="front_right_d_contact_link">
-    <inertial>
-      <mass value="0.01" />
-      <origin xyz="0 0 0" />
-      <inertia ixx="1e-5" ixy="0" ixz="0" iyy="1e-5" iyz="0" izz="1e-5" />
-    </inertial>
-    <visual>
-      <origin xyz="0 -0.05 0" rpy="${pi/2} 0 0" />
-      <geometry>
-        <cylinder radius="0.018" length="0.19" />
-      </geometry>
-      <material name="grey">
-        <color rgba="0.5 0.5 0.5 1" />
-      </material>
-    </visual>
-    <collision>
-      <origin xyz="0 -0.05 0" rpy="${pi/2} 0 0" />
-      <geometry>
-        <cylinder radius="0.018" length="0.19" />
-      </geometry>
-    </collision>
-  </link>
-  <joint name="front_right_d_contact_joint" type="fixed">
-    <parent link="front_right_d" /> <!-- Nombre del link actual de la pata -->
-    <child link="front_right_d_contact_link" />
-    <origin xyz="0.4 0 0" rpy="0 0 0" /> <!-- Ajusta la posición al final de la pata -->
-  </joint>
-  <link name="back_right_d_contact_link">
-    <inertial>
-      <mass value="0.01" />
-      <origin xyz="0 0 0" />
-      <inertia ixx="1e-5" ixy="0" ixz="0" iyy="1e-5" iyz="0" izz="1e-5" />
-    </inertial>
-    <visual>
-      <origin xyz="0 0.05 0" rpy="${pi/2} 0 0" />
-      <geometry>
-        <cylinder radius="0.018" length="0.19" />
-      </geometry>
-      <material name="grey">
-        <color rgba="0.5 0.5 0.5 1" />
-      </material>
-    </visual>
-    <collision>
-      <origin xyz="0 0.05 0" rpy="${pi/2} 0 0" />
-      <geometry>
-        <cylinder radius="0.018" length="0.19" />
-      </geometry>
-    </collision>
-  </link>
-  <joint name="back_right_d_contact_joint" type="fixed">
-    <parent link="back_right_d" /> <!-- Nombre del link actual de la pata -->
-    <child link="back_right_d_contact_link" />
-    <origin xyz="0.4 0 0" rpy="0 0 0" /> <!-- Ajusta la posición al final de la pata -->
-  </joint>
-   <link name="back_left_d_contact_link">
-    <inertial>
-      <mass value="0.01" />
-      <origin xyz="0 0 0" />
-      <inertia ixx="1e-5" ixy="0" ixz="0" iyy="1e-5" iyz="0" izz="1e-5" />
-    </inertial>
-    <visual>
-      <origin xyz="0 -0.05 0" rpy="${pi/2} 0 0" />
-      <geometry>
-        <cylinder radius="0.018" length="0.19" />
-      </geometry>
-      <material name="grey">
-        <color rgba="0.5 0.5 0.5 1" />
-      </material>
-    </visual>
-    <collision>
-      <origin xyz="0 -0.05 0" rpy="${pi/2} 0 0" />
-      <geometry>
-        <cylinder radius="0.018" length="0.19" />
-      </geometry>
-    </collision>
-  </link>
-  <joint name="back_left_d_contact_joint" type="fixed">
-    <parent link="back_left_d" /> <!-- Nombre del link actual de la pata -->
-    <child link="back_left_d_contact_link" />
-    <origin xyz="0.4 0 0" rpy="0 0 0" /> <!-- Ajusta la posición al final de la pata -->
-  </joint>
 </robot>

File: quadruped_description/urdf/quadruped_robot3.urdf.xacro (robot description, xacro)
@@ -5,15 +5,8 @@
   <link name="body">
     <inertial>
-      <origin rpy="0 ${pi /8} 0" xyz="0 0 0.05"/>
-      <mass
-        value="15" />
-      <!-- <inertia
-        ixx="0.04" ixy="-0.000009" ixz="0.0045"
-        iyy="0.043" iyz="-0.000022"
-        izz="0.03" /> -->
-      <inertia
-        ixx="0.08" ixy="-0.0000173" ixz="0.00929"
-        iyy="0.08613" iyz="-0.0000446"
-        izz="0.0601" />
+      <mass value="1" />
+      <inertia ixx="1" ixy="0"  ixz="0"
+               iyy="1" iyz="0"
+               izz="1" />
     </inertial>
     <visual>
@@ -69,11 +62,8 @@
   <link name="front_left_u">
     <inertial>
-      <mass value="0.8" />
-      <!-- <inertia ixx="0.00025" ixy="0.0012"  ixz="0.0"
-               iyy="0.022" iyz="0.0"
-               izz="0.022" /> -->
-      <inertia ixx="0.00051" ixy="0.0025"  ixz="0.0"
-               iyy="0.044" iyz="0.0"
-               izz="0.044" />
+      <mass value="1" />
+      <inertia ixx="1" ixy="0"  ixz="0"
+               iyy="1" iyz="0"
+               izz="1" />
     </inertial>
     <visual>
@@ -95,11 +85,8 @@
   <link name="front_right_u">
     <inertial>
-      <mass value="0.8" />
-      <!-- <inertia ixx="0.00035" ixy="-0.0019"  ixz="0.0"
-               iyy="0.022" iyz="0.0"
-               izz="0.022" /> -->
-      <inertia ixx="0.00076" ixy="-0.00385"  ixz="0.0"
-               iyy="0.044" iyz="0.0"
-               izz="0.044" />
+      <mass value="1" />
+      <inertia ixx="1" ixy="0"  ixz="0"
+               iyy="1" iyz="0"
+               izz="1" />
     </inertial>
     <visual>
@@ -121,11 +108,8 @@
   <link name="back_left_u">
     <inertial>
-      <mass value="0.8" />
-      <!-- <inertia ixx="0.00035" ixy="-0.0019"  ixz="0.0"
-               iyy="0.022" iyz="0.0"
-               izz="0.022" /> -->
-      <inertia ixx="0.00076" ixy="-0.00385"  ixz="0.0"
-               iyy="0.044" iyz="0.0"
-               izz="0.044" />
+      <mass value="1" />
+      <inertia ixx="1" ixy="0"  ixz="0"
+               iyy="1" iyz="0"
+               izz="1" />
     </inertial>
     <visual>
@@ -147,11 +131,8 @@
   <link name="back_right_u">
     <inertial>
-      <mass value="0.8" />
-      <!-- <inertia ixx="0.00025" ixy="0.0012"  ixz="0.0"
-               iyy="0.022" iyz="0.0"
-               izz="0.022" /> -->
-      <inertia ixx="0.00051" ixy="0.0025"  ixz="0.0"
-               iyy="0.044" iyz="0.0"
-               izz="0.044" />
+      <mass value="1" />
+      <inertia ixx="1" ixy="0"  ixz="0"
+               iyy="1" iyz="0"
+               izz="1" />
     </inertial>
     <visual>
@@ -173,14 +154,8 @@
   <link name="front_left_d">
     <inertial>
-      <mass value="1.0" />
-      <!-- <inertia ixx="0.0039" ixy="0.012"  ixz="0.0"
-               iyy="0.1412" iyz="0.0"
-               izz="0.1447" /> Pata nueva-->
-      <!-- <inertia ixx="0.000045" ixy="0.0019"  ixz="0.0"
-               iyy="0.022" iyz="0.0"
-               izz="0.022" /> -->
-      <inertia ixx="0.0009" ixy="0.0038"  ixz="0.0"
-               iyy="0.044" iyz="0.0"
-               izz="0.0457" />
+      <mass value="1" />
+      <inertia ixx="1" ixy="0"  ixz="0"
+               iyy="1" iyz="0"
+               izz="1" />
     </inertial>
     <visual>
@@ -202,11 +177,8 @@
   <link name="front_right_d">
     <inertial>
-      <mass value="1.0" />
-      <!-- <inertia ixx="0.000045" ixy="-0.0019"  ixz="0.0"
-               iyy="0.022" iyz="0.0"
-               izz="0.022" /> -->
-      <inertia ixx="0.0009" ixy="-0.0038"  ixz="0.0"
-               iyy="0.044" iyz="0.0"
-               izz="0.0457" />
+      <mass value="1" />
+      <inertia ixx="1" ixy="0"  ixz="0"
+               iyy="1" iyz="0"
+               izz="1" />
     </inertial>
     <visual>
@@ -228,11 +200,8 @@
   <link name="back_left_d">
     <inertial>
-      <mass value="1.0" />
-      <!-- <inertia ixx="0.000045" ixy="-0.0019"  ixz="0.0"
-               iyy="0.022" iyz="0.0"
-               izz="0.022" /> -->
-      <inertia ixx="0.0009" ixy="-0.0038"  ixz="0.0"
-               iyy="0.044" iyz="0.0"
-               izz="0.0457" />
+      <mass value="1" />
+      <inertia ixx="1" ixy="0"  ixz="0"
+               iyy="1" iyz="0"
+               izz="1" />
     </inertial>
     <visual>
@@ -254,11 +223,8 @@
   <link name="back_right_d">
     <inertial>
-      <mass value="1.0" />
-      <!-- <inertia ixx="0.000045" ixy="0.0019"  ixz="0.0"
-               iyy="0.022" iyz="0.0"
-               izz="0.022" /> -->
-      <inertia ixx="0.0009" ixy="0.0038"  ixz="0.0"
-               iyy="0.044" iyz="0.0"
-               izz="0.0457" />
+      <mass value="1" />
+      <inertia ixx="1" ixy="0"  ixz="0"
+               iyy="1" iyz="0"
+               izz="1" />
     </inertial>
     <visual>
