Commit message: Se mejoro las inercias del cuadrupedo diferenciando entre los links de izqueirda y derecha

File: quadruped_description/urdf/quadruped_robot.urdf.xacro (robot description, xacro)
@@ -65,7 +65,7 @@
     <inertial>
       <mass value="0.8" />
-      <inertia ixx="0.0008" ixy="0.0063"  ixz="0.0"
-               iyy="0.07" iyz="0.0"
-               izz="0.071" />
+      <inertia ixx="0.00051" ixy="0.0025"  ixz="0.0"
+               iyy="0.044" iyz="0.0"
+               izz="0.044" />
     </inertial>
     <visual>
@@ -88,7 +88,7 @@
     <inertial>
       <mass value="0.8" />
-      <inertia ixx="0.0008" ixy="0.0063"  ixz="0.0"
-               iyy="0.07" iyz="0.0"
-               izz="0.071" />
+      <inertia ixx="0.00076" ixy="-0.00385"  ixz="0.0"
+               iyy="0.044" iyz="0.0"
+               izz="0.044" />
     </inertial>
     <visual>
@@ -111,7 +111,7 @@
     <inertial>
       <mass value="0.8" />
-      <inertia ixx="0.0008" ixy="0.0063"  ixz="0.0"
-               iyy="0.07" iyz="0.0"
-               izz="0.071" />
+      <inertia ixx="0.00076" ixy="-0.00385"  ixz="0.0"
+               iyy="0.044" iyz="0.0"
+               izz="0.044" />
     </inertial>
     <visual>
@@ -134,7 +134,7 @@
     <inertial>
       <mass value="0.8" />
-      <inertia ixx="0.0008" ixy="0.0063"  ixz="0.0"
-               iyy="0.07" iyz="0.0"
-               izz="0.071" />
+      <inertia ixx="0.00051" ixy="0.0025"  ixz="0.0"
+               iyy="0.044" iyz="0.0"
+               izz="0.044" />
     </inertial>
     <visual>
@@ -157,7 +157,10 @@
     <inertial>
       <mass value="1.0" />
-      <inertia ixx="0.0039" ixy="0.012"  ixz="0.0"
+      <!-- <inertia ixx="0.0039" ixy="0.012"  ixz="0.0"
                iyy="0.1412" iyz="0.0"
-               izz="0.1447" />
+               izz="0.1447" /> Pata nueva-->
+      <inertia ixx="0.0009" ixy="0.0038"  ixz="0.0"
+               iyy="0.044" iyz="0.0"
+               izz="0.0457" />
     </inertial>
     <visual>
@@ -180,7 +183,7 @@
     <inertial>
       <mass value="1.0" />
-      <inertia ixx="0.0039" ixy="0.012"  ixz="0.0"
-               iyy="0.1412" iyz="0.0"
-               izz="0.1447" />
+      <inertia ixx="0.0009" ixy="-0.0038"  ixz="0.0"
+               iyy="0.044" iyz="0.0"
+               izz="0.0457" />
     </inertial>
     <visual>
@@ -203,7 +206,7 @@
     <inertial>
       <mass value="1.0" />
-      <inertia ixx="0.0039" ixy="0.012"  ixz="0.0"
-               iyy="0.1412" iyz="0.0"
-               izz="0.1447" />
+      <inertia ixx="0.0009" ixy="-0.0038"  ixz="0.0"
+               iyy="0.044" iyz="0.0"
+               izz="0.0457" />
     </inertial>
     <visual>
@@ -226,7 +229,7 @@
     <inertial>
       <mass value="1.0" />
-      <inertia ixx="0.0039" ixy="0.012"  ixz="0.0"
-               iyy="0.1412" iyz="0.0"
-               izz="0.1447" />
+      <inertia ixx="0.0009" ixy="0.0038"  ixz="0.0"
+               iyy="0.044" iyz="0.0"
+               izz="0.0457" />
     </inertial>
     <visual>

Commit message: Se quitan los cntactos en las patas del urdf

File: quadruped_description/urdf/quadruped_robot.urdf.xacro (robot description, xacro)
@@ -355,111 +355,3 @@
     <axis xyz="0 1 0" />
   </joint>
-  <link name="front_left_d_contact_link">
-    <inertial>
-      <mass value="0.01" />
-      <origin xyz="0 0 0" />
-      <inertia ixx="1e-5" ixy="0" ixz="0" iyy="1e-5" iyz="0" izz="1e-5" />
-    </inertial>
-    <!-- <visual>
-      <origin xyz="0 0.05 0" rpy="${pi/2} 0 0" />
-      <geometry>
-        <cylinder radius="0.018" length="0.19" />
-      </geometry>
-      <material name="grey">
-        <color rgba="0.5 0.5 0.5 1" />
-      </material>
-    </visual> -->
-    <collision>
-      <origin xyz="0 0.05 0" rpy="${pi/2} 0 0" />
-      <geometry>
-        <cylinder radius="0.018" length="0.19" />
-      </geometry>
-    </collision>
-  </link>
-  <joint name="front_left_d_contact_joint" type="fixed">
-    <parent link="front_left_d" /> <!-- Nombre del link actual de la pata -->
-    <child link="front_left_d_contact_link" />
-    <origin xyz="0.4 0 0" rpy="0 0 0" /> <!-- Ajusta la posición al final de la pata -->
-  </joint>
-  <link name="front_right_d_contact_link">
-    <inertial>
-      <mass value="0.01" />
-      <origin xyz="0 0 0" />
-      <inertia ixx="1e-5" ixy="0" ixz="0" iyy="1e-5" iyz="0" izz="1e-5" />
-    </inertial>
-    <!-- <visual>
-      <origin xyz="0 -0.05 0" rpy="${pi/2} 0 0" />
-      <geometry>
-        <cylinder radius="0.018" length="0.19" />
-      </geometry>
-      <material name="grey">
-        <color rgba="0.5 0.5 0.5 1" />
-      </material>
-    </visual> -->
-    <collision>
-      <origin xyz="0 -0.05 0" rpy="${pi/2} 0 0" />
-      <geometry>
-        <cylinder radius="0.018" length="0.19" />
-      </geometry>
-    </collision>
-  </link>
-  <joint name="front_right_d_contact_joint" type="fixed">
-    <parent link="front_right_d" /> <!-- Nombre del link actual de la pata -->
-    <child link="front_right_d_contact_link" />
-    <origin xyz="0.4 0 0" rpy="0 0 0" /> <!-- Ajusta la posición al final de la pata -->
-  </joint>
-  <link name="back_right_d_contact_link">
-    <inertial>
-      <mass value="0.01" />
-      <origin xyz="0 0 0" />
-      <inertia ixx="1e-5" ixy="0" ixz="0" iyy="1e-5" iyz="0" izz="1e-5" />
-    </inertial>
-    <!-- <visual>
-      <origin xyz="0 0.05 0" rpy="${pi/2} 0 0" />
-      <geometry>
-        <cylinder radius="0.018" length="0.19" />
-      </geometry>
-      <material name="grey">
-        <color rgba="0.5 0.5 0.5 1" />
-      </material>
-    </visual> -->
-    <collision>
-      <origin xyz="0 0.05 0" rpy="${pi/2} 0 0" />
-      <geometry>
-        <cylinder radius="0.018" length="0.19" />
-      </geometry>
-    </collision>
-  </link>
-  <joint name="back_right_d_contact_joint" type="fixed">
-    <parent link="back_right_d" /> <!-- Nombre del link actual de la pata -->
-    <child link="back_right_d_contact_link" />
-    <origin xyz="0.4 0 0" rpy="0 0 0" /> <!-- Ajusta la posición al final de la pata -->
-  </joint>
-   <link name="back_left_d_contact_link">
-    <inertial>
-      <mass value="0.01" />
-      <origin xyz="0 0 0" />
-      <inertia ixx="1e-5" ixy="0" ixz="0" iyy="1e-5" iyz="0" izz="1e-5" />
-    </inertial>
-    <!-- <visual>
-      <origin xyz="0 -0.05 0" rpy="${pi/2} 0 0" />
-      <geometry>
-        <cylinder radius="0.018" length="0.19" />
-      </geometry>
-      <material name="grey">
-        <color rgba="0.5 0.5 0.5 1" />
-      </material>
-    </visual> -->
-    <collision>
-      <origin xyz="0 -0.05 0" rpy="${pi/2} 0 0" />
-      <geometry>
-        <cylinder radius="0.018" length="0.19" />
-      </geometry>
-    </collision>
-  </link>
-  <joint name="back_left_d_contact_joint" type="fixed">
-    <parent link="back_left_d" /> <!-- Nombre del link actual de la pata -->
-    <child link="back_left_d_contact_link" />
-    <origin xyz="0.4 0 0" rpy="0 0 0" /> <!-- Ajusta la posición al final de la pata -->
-  </joint>
 </robot>
