Commit message: Ya se pulican los controladores de manera exitosa en gazebo

File: quadruped_description/urdf/quadruped_gazebo.urdf.xacro (robot description, xacro)
@@ -14,5 +14,14 @@
       </state_interface>
       <state_interface name="velocity" />
-      <state_interface name="effort" />
+    </joint>
+    <joint name="front_right_joint1">
+      <command_interface name="position">
+        <param name="min">-3.14</param>
+        <param name="max">3.14</param>
+      </command_interface>
+      <state_interface name="position">
+        <param name="initial_value">0</param>
+      </state_interface>
+      <state_interface name="velocity" />
     </joint>
   </ros2_control>
@@ -20,5 +29,5 @@
   <gazebo>
     <plugin name="gazebo_ros2_control" filename="libgazebo_ros2_control.so">
-      <parameters>$(find quadruped_gazebo)/config/joint_controller.yaml</parameters>
+      <parameters>/home/erick/quad_ws/src/quadruped_description/config/joint_controller.yaml</parameters>
     </plugin>
   </gazebo>

File: quadruped_description/urdf/quadruped_robot.urdf.xacro (robot description, xacro)
@@ -18,5 +18,5 @@
       <origin rpy="0 0 ${pi / 2.0}" xyz="0 0 -0.06"/>
       <geometry>
-        <mesh filename="model://my_quadruped/meshes/frame_aluminum_motor.stl" />
+        <mesh filename="file://$(find quadruped_description)/meshes/frame_aluminum_motor.stl" />
       </geometry>
       <material name="grey"/>
@@ -27,5 +27,5 @@
         rpy="0 0 ${pi / 2.0}" />
       <geometry>
-        <mesh filename="model://my_quadruped/meshes/frame_aluminum_motor.stl" />
+        <mesh filename="file://$(find quadruped_description)//meshes/frame_aluminum_motor.stl" />
       </geometry>
     </collision>
@@ -54,5 +54,5 @@
       <geometry>
         <mesh
-          filename="model://my_quadruped/meshes/camera_link.stl" />
+          filename="file://$(find quadruped_description)//meshes/camera_link.stl" />
       </geometry>
       <material
@@ -68,5 +68,5 @@
       <geometry>
         <mesh
-          filename="model://my_quadruped/meshes/camera_link.stl" />
+          filename="file://$(find quadruped_description)//meshes/camera_link.stl" />
       </geometry>
     </collision>
@@ -99,5 +99,5 @@
       <origin rpy="1.57 0 1.57" xyz="0 0 0"/>
       <geometry>
-        <mesh filename="model://my_quadruped/meshes/joint_gear_upper_assembly.stl" />
+        <mesh filename="file://$(find quadruped_description)//meshes/joint_gear_upper_assembly.stl" />
       </geometry>
       <material name="grey"/>
@@ -108,5 +108,5 @@
         rpy="1.57 0 1.57" />
       <geometry>
-        <mesh filename="model://my_quadruped/meshes/joint_gear_upper_assembly.stl" />
+        <mesh filename="file://$(find quadruped_description)//meshes/joint_gear_upper_assembly.stl" />
       </geometry>
     </collision>
@@ -129,5 +129,5 @@
       <origin rpy="1.57 3.14 1.57" xyz="0 0 0"/>
       <geometry>
-        <mesh filename="model://my_quadruped/meshes/joint_gear_upper_assembly.stl" />
+        <mesh filename="file://$(find quadruped_description)//meshes/joint_gear_upper_assembly.stl" />
       </geometry>
       <material name="grey"/>
@@ -138,5 +138,5 @@
         rpy="1.57 3.14 1.57" />
       <geometry>
-        <mesh filename="model://my_quadruped/meshes/joint_gear_upper_assembly.stl" />
+        <mesh filename="file://$(find quadruped_description)//meshes/joint_gear_upper_assembly.stl" />
       </geometry>
     </collision>
@@ -152,5 +152,5 @@
       <origin rpy="1.57 3.14 1.57" xyz="0 0 0"/>
       <geometry>
-        <mesh filename="model://my_quadruped/meshes/joint_gear_upper_assembly.stl" />
+        <mesh filename="file://$(find quadruped_description)//meshes/joint_gear_upper_assembly.stl" />
       </geometry>
       <material name="grey"/>
@@ -161,5 +161,5 @@
         rpy="1.57 3.14 1.57" />
       <geometry>
-        <mesh filename="model://my_quadruped/meshes/joint_gear_upper_assembly.stl" />
+        <mesh filename="file://$(find quadruped_description)//meshes/joint_gear_upper_assembly.stl" />
       </geometry>
     </collision>
@@ -175,5 +175,5 @@
       <origin rpy="1.57 0 1.57" xyz="0 0 0"/>
       <geometry>
-        <mesh filename="model://my_quadruped/meshes/joint_gear_upper_assembly.stl" />
+        <mesh filename="file://$(find quadruped_description)//meshes/joint_gear_upper_assembly.stl" />
       </geometry>
       <material name="grey"/>
@@ -184,5 +184,5 @@
         rpy="1.57 0 1.57" />
       <geometry>
-        <mesh filename="model://my_quadruped/meshes/joint_gear_upper_assembly.stl" />
+        <mesh filename="file://$(find quadruped_description)//meshes/joint_gear_upper_assembly.stl" />
       </geometry>
     </collision>
@@ -198,5 +198,5 @@
       <origin rpy="1.57 0 1.57" xyz="0 0 0"/>
       <geometry>
-        <mesh filename="model://my_quadruped/meshes/Assembly_lower_link_v2.stl" />
+        <mesh filename="file://$(find quadruped_description)//meshes/Assembly_lower_link_v2.stl" />
       </geometry>
       <material name="grey"/>
@@ -207,5 +207,5 @@
         rpy="1.57 0 1.57" />
       <geometry>
-        <mesh filename="model://my_quadruped/meshes/Assembly_lower_link_v2.stl" />
+        <mesh filename="file://$(find quadruped_description)//meshes/Assembly_lower_link_v2.stl" />
       </geometry>
     </collision>
@@ -221,5 +221,5 @@
       <origin rpy="-1.57 0 -1.57" xyz="0 0 0"/>
       <geometry>
-        <mesh filename="model://my_quadruped/meshes/Assembly_lower_link_v2.stl" />
+        <mesh filename="file://$(find quadruped_description)//meshes/Assembly_lower_link_v2.stl" />
       </geometry>
       <material name="grey"/>
@@ -230,5 +230,5 @@
         rpy="-1.57 0 -1.57" />
       <geometry>
-        <mesh filename="model://my_quadruped/meshes/Assembly_lower_link_v2.stl" />
+        <mesh filename="file://$(find quadruped_description)//meshes/Assembly_lower_link_v2.stl" />
       </geometry>
     </collision>
@@ -244,5 +244,5 @@
       <origin rpy="-1.57 0 -1.57" xyz="0 0 0"/>
       <geometry>
-        <mesh filename="model://my_quadruped/meshes/Assembly_lower_link_v2.stl" />
+        <mesh filename="file://$(find quadruped_description)//meshes/Assembly_lower_link_v2.stl" />
       </geometry>
       <material name="grey"/>
@@ -253,5 +253,5 @@
         rpy="-1.57 0 -1.57" />
       <geometry>
-        <mesh filename="model://my_quadruped/meshes/Assembly_lower_link_v2.stl" />
+        <mesh filename="file://$(find quadruped_description)//meshes/Assembly_lower_link_v2.stl" />
       </geometry>
     </collision>
@@ -267,5 +267,5 @@
       <origin rpy="1.57 0 1.57" xyz="0 0 0"/>
       <geometry>
-        <mesh filename="model://my_quadruped/meshes/Assembly_lower_link_v2.stl" />
+        <mesh filename="file://$(find quadruped_description)//meshes/Assembly_lower_link_v2.stl" />
       </geometry>
       <material name="grey"/>
@@ -276,5 +276,5 @@
         rpy="1.57 0 1.57" />
       <geometry>
-        <mesh filename="model://my_quadruped/meshes/Assembly_lower_link_v2.stl" />
+        <mesh filename="file://$(find quadruped_description)//meshes/Assembly_lower_link_v2.stl" />
       </geometry>
     </collision>

Commit message: Se arreglo las inercias del quadrupedo en el archivo .xacro de manera que no salga volando en gazebo, ademas se anadio un archivo stl para la nueva pata

File: quadruped_description/urdf/quadruped_gazebo.urdf.xacro (robot description, xacro)
@@ -11,9 +11,79 @@
       </command_interface>
       <state_interface name="position">
+        <param name="initial_value">1.0</param>
+      </state_interface>
+      <state_interface name="velocity" />
+    </joint>
+    <joint name="front_right_joint1">
+      <command_interface name="position">
+        <param name="min">-3.14</param>
+        <param name="max">3.14</param>
+      </command_interface>
+      <state_interface name="position">
         <param name="initial_value">0</param>
       </state_interface>
       <state_interface name="velocity" />
     </joint>
-    <joint name="front_right_joint1">
+    <joint name="front_right_joint2">
+      <command_interface name="position">
+        <param name="min">-3.14</param>
+        <param name="max">3.14</param>
+      </command_interface>
+      <state_interface name="position">
+        <param name="initial_value">0</param>
+      </state_interface>
+      <state_interface name="velocity" />
+    </joint>
+    <joint name="front_left_joint1">
+      <command_interface name="position">
+        <param name="min">-3.14</param>
+        <param name="max">3.14</param>
+      </command_interface>
+      <state_interface name="position">
+        <param name="initial_value">0</param>
+      </state_interface>
+      <state_interface name="velocity" />
+    </joint>
+    <joint name="front_left_joint2">
+      <command_interface name="position">
+        <param name="min">-3.14</param>
+        <param name="max">3.14</param>
+      </command_interface>
+      <state_interface name="position">
+        <param name="initial_value">0</param>
+      </state_interface>
+      <state_interface name="velocity" />
+    </joint>
+    <joint name="back_left_joint1">
+      <command_interface name="position">
+        <param name="min">-3.14</param>
+        <param name="max">3.14</param>
+      </command_interface>
+      <state_interface name="position">
+        <param name="initial_value">0</param>
+      </state_interface>
+      <state_interface name="velocity" />
+    </joint>
+    <joint name="back_left_joint2">
+      <command_interface name="position">
+        <param name="min">-3.14</param>
+        <param name="max">3.14</param>
+      </command_interface>
+      <state_interface name="position">
+        <param name="initial_value">0</param>
+      </state_interface>
+      <state_interface name="velocity" />
+    </joint>
+    <joint name="back_right_joint1">
+      <command_interface name="position">
+        <param name="min">-3.14</param>
+        <param name="max">3.14</param>
+      </command_interface>
+      <state_interface name="position">
+        <param name="initial_value">0</param>
+      </state_interface>
+      <state_interface name="velocity" />
+    </joint>
+    <joint name="back_right_joint2">
       <command_interface name="position">
         <param name="min">-3.14</param>

File: quadruped_description/urdf/quadruped_robot.urdf.xacro (robot description, xacro)
@@ -6,12 +6,9 @@
     <inertial>
       <mass
-        value="3.0416" />
+        value="3" />
       <inertia
-        ixx="0.0073301"
-        ixy="2.1671E-09"
-        ixz="1.9602E-06"
-        iyy="0.0077176"
-        iyz="-1.1292E-05"
-        izz="0.0059691" />
+        ixx="0.039" ixy="-0.0000173" ixz="0.00929"
+        iyy="0.04613" iyz="-0.0000446"
+        izz="0.0301" />
     </inertial>
     <visual>
@@ -31,20 +28,13 @@
     </collision>
   </link>
-  <joint name="dummy_joint" type="fixed">
-     <parent link="dummy"/>
-     <child link="body"/>
-  </joint>
   <link
     name="camera_link">
     <inertial>
       <mass
-        value="0.046222" />
+        value="0.05" />
       <inertia
-        ixx="2.633E-06"
-        ixy="-4.2166E-09"
-        ixz="1.2531E-08"
-        iyy="2.5049E-05"
-        iyz="9.9718E-08"
-        izz="2.639E-05" />
+        ixx="0.0000275" ixy="0.000000153" ixz="0.0"
+        iyy="0.0000867" iyz="0.0"
+        izz="0.000110" />
     </inertial>
     <visual>
@@ -72,4 +62,192 @@
     </collision>
   </link>
+  <link name="front_left_u">
+    <inertial>
+      <mass value="0.8" />
+      <inertia ixx="0.0008" ixy="0.0063"  ixz="0.0"
+               iyy="0.07" iyz="0.0"
+               izz="0.071" />
+    </inertial>
+    <visual>
+      <origin rpy="1.57 0 1.57" xyz="0 0 0"/>
+      <geometry>
+        <mesh filename="file://$(find quadruped_description)//meshes/joint_gear_upper_assembly.stl" />
+      </geometry>
+      <material name="grey"/>
+    </visual>
+    <collision>
+      <origin
+        xyz="0 0 0"
+        rpy="1.57 0 1.57" />
+      <geometry>
+        <mesh filename="file://$(find quadruped_description)//meshes/joint_gear_upper_assembly.stl" />
+      </geometry>
+    </collision>
+  </link>
+  <link name="front_right_u">
+    <inertial>
+      <mass value="0.8" />
+      <inertia ixx="0.0008" ixy="0.0063"  ixz="0.0"
+               iyy="0.07" iyz="0.0"
+               izz="0.071" />
+    </inertial>
+    <visual>
+      <origin rpy="1.57 3.14 1.57" xyz="0 0 0"/>
+      <geometry>
+        <mesh filename="file://$(find quadruped_description)//meshes/joint_gear_upper_assembly.stl" />
+      </geometry>
+      <material name="grey"/>
+    </visual>
+    <collision>
+      <origin
+        xyz="0 0 0"
+        rpy="1.57 3.14 1.57" />
+      <geometry>
+        <mesh filename="file://$(find quadruped_description)//meshes/joint_gear_upper_assembly.stl" />
+      </geometry>
+    </collision>
+  </link>
+  <link name="back_left_u">
+    <inertial>
+      <mass value="0.8" />
+      <inertia ixx="0.0008" ixy="0.0063"  ixz="0.0"
+               iyy="0.07" iyz="0.0"
+               izz="0.071" />
+    </inertial>
+    <visual>
+      <origin rpy="1.57 3.14 1.57" xyz="0 0 0"/>
+      <geometry>
+        <mesh filename="file://$(find quadruped_description)//meshes/joint_gear_upper_assembly.stl" />
+      </geometry>
+      <material name="grey"/>
+    </visual>
+    <collision>
+      <origin
+        xyz="0 0 0"
+        rpy="1.57 3.14 1.57" />
+      <geometry>
+        <mesh filename="file://$(find quadruped_description)//meshes/joint_gear_upper_assembly.stl" />
+      </geometry>
+    </collision>
+  </link>
+  <link name="back_right_u">
+    <inertial>
+      <mass value="0.8" />
+      <inertia ixx="0.0008" ixy="0.0063"  ixz="0.0"
+               iyy="0.07" iyz="0.0"
+               izz="0.071" />
+    </inertial>
+    <visual>
+      <origin rpy="1.57 0 1.57" xyz="0 0 0"/>
+      <geometry>
+        <mesh filename="file://$(find quadruped_description)//meshes/joint_gear_upper_assembly.stl" />
+      </geometry>
+      <material name="grey"/>
+    </visual>
+    <collision>
+      <origin
+        xyz="0 0 0"
+        rpy="1.57 0 1.57" />
+      <geometry>
+        <mesh filename="file://$(find quadruped_description)//meshes/joint_gear_upper_assembly.stl" />
+      </geometry>
+    </collision>
+  </link>
+  <link name="front_left_d">
+    <inertial>
+      <mass value="1.0" />
+      <inertia ixx="0.0039" ixy="0.012"  ixz="0.0"
+               iyy="0.1412" iyz="0.0"
+               izz="0.1447" />
+    </inertial>
+    <visual>
+      <origin rpy="1.57 0 1.57" xyz="0 0 0"/>
+      <geometry>
+        <mesh filename="file://$(find quadruped_description)//meshes/Assembly_lower_link_v2.stl" />
+      </geometry>
+      <material name="grey"/>
+    </visual>
+    <collision>
+      <origin
+        xyz="0 0 0"
+        rpy="1.57 0 1.57" />
+      <geometry>
+        <mesh filename="file://$(find quadruped_description)//meshes/Assembly_lower_link_v2.stl" />
+      </geometry>
+    </collision>
+  </link>
+  <link name="front_right_d">
+    <inertial>
+      <mass value="1.0" />
+      <inertia ixx="0.0039" ixy="0.012"  ixz="0.0"
+               iyy="0.1412" iyz="0.0"
+               izz="0.1447" />
+    </inertial>
+    <visual>
+      <origin rpy="-1.57 0 -1.57" xyz="0 0 0"/>
+      <geometry>
+        <mesh filename="file://$(find quadruped_description)//meshes/Assembly_lower_link_v2.stl" />
+      </geometry>
+      <material name="grey"/>
+    </visual>
+    <collision>
+      <origin
+        xyz="0 0 0"
+        rpy="-1.57 0 -1.57" />
+      <geometry>
+        <mesh filename="file://$(find quadruped_description)//meshes/Assembly_lower_link_v2.stl" />
+      </geometry>
+    </collision>
+  </link>
+  <link name="back_left_d">
+    <inertial>
+      <mass value="1.0" />
+      <inertia ixx="0.0039" ixy="0.012"  ixz="0.0"
+               iyy="0.1412" iyz="0.0"
+               izz="0.1447" />
+    </inertial>
+    <visual>
+      <origin rpy="-1.57 0 -1.57" xyz="0 0 0"/>
+      <geometry>
+        <mesh filename="file://$(find quadruped_description)//meshes/Assembly_lower_link_v2.stl" />
+      </geometry>
+      <material name="grey"/>
+    </visual>
+    <collision>
+      <origin
+        xyz="0 0 0"
+        rpy="-1.57 0 -1.57" />
+      <geometry>
+        <mesh filename="file://$(find quadruped_description)//meshes/Assembly_lower_link_v2.stl" />
+      </geometry>
+    </collision>
+  </link>
+  <link name="back_right_d">
+    <inertial>
+      <mass value="1.0" />
+      <inertia ixx="0.0039" ixy="0.012"  ixz="0.0"
+               iyy="0.1412" iyz="0.0"
+               izz="0.1447" />
+    </inertial>
+    <visual>
+      <origin rpy="1.57 0 1.57" xyz="0 0 0"/>
+      <geometry>
+        <mesh filename="file://$(find quadruped_description)//meshes/Assembly_lower_link_v2.stl" />
+      </geometry>
+      <material name="grey"/>
+    </visual>
+    <collision>
+      <origin
+        xyz="0 0 0"
+        rpy="1.57 0 1.57" />
+      <geometry>
+        <mesh filename="file://$(find quadruped_description)//meshes/Assembly_lower_link_v2.stl" />
+      </geometry>
+    </collision>
+  </link>
+  <joint name="dummy_joint" type="fixed">
+     <parent link="dummy"/>
+     <child link="body"/>
+  </joint>
   <joint
     name="camera_joint" type="revolute">
@@ -89,27 +267,18 @@
       velocity="100" />
   </joint>
-  <link name="front_left_u">
-    <inertial>
-      <mass value="0.814" />
-      <inertia ixx="0.008" ixy="0.0"  ixz="0.001"
-               iyy="0.008" iyz="0.001"
-               izz="0.001" />
-    </inertial>
-    <visual>
-      <origin rpy="1.57 0 1.57" xyz="0 0 0"/>
-      <geometry>
-        <mesh filename="file://$(find quadruped_description)//meshes/joint_gear_upper_assembly.stl" />
-      </geometry>
-      <material name="grey"/>
-    </visual>
-    <collision>
-      <origin
-        xyz="0 0 0"
-        rpy="1.57 0 1.57" />
-      <geometry>
-        <mesh filename="file://$(find quadruped_description)//meshes/joint_gear_upper_assembly.stl" />
-      </geometry>
-    </collision>
-  </link>
+    <joint name="front_right_joint1" type="revolute">
+    <limit effort="1000.0" lower="-3.14" upper="3.14" velocity="0.5"/>
+    <parent link="body"/>
+    <child link="front_right_u"/>
+    <origin xyz="0.11 -0.05 0" rpy="0 0 0" />
+    <axis xyz="0 1 0" />
+  </joint>
+  <joint name="front_right_joint2" type="revolute">
+    <limit effort="1000.0" lower="-3.14" upper="3.14" velocity="0.5"/>
+    <parent link="front_right_u"/>
+    <child link="front_right_d"/>
+    <origin xyz="0.4 -0.005 0" rpy="0 0 0" />
+    <axis xyz="0 1 0" />
+  </joint>
   <joint name="front_left_joint1" type="revolute">
     <limit effort="1000.0" lower="-3.14" upper="3.14" velocity="0.5"/>
@@ -119,179 +288,4 @@
     <axis xyz="0 1 0" />
   </joint>
-  <link name="front_right_u">
-    <inertial>
-      <mass value="0.814" />
-      <inertia ixx="7701247.352E-09" ixy="96047.710E-09"  ixz="-1228944.675E-09"
-               iyy="7801785.041E-09" iyz="550113.749E-09"
-               izz="877983.793E-09" />
-    </inertial>
-    <visual>
-      <origin rpy="1.57 3.14 1.57" xyz="0 0 0"/>
-      <geometry>
-        <mesh filename="file://$(find quadruped_description)//meshes/joint_gear_upper_assembly.stl" />
-      </geometry>
-      <material name="grey"/>
-    </visual>
-    <collision>
-      <origin
-        xyz="0 0 0"
-        rpy="1.57 3.14 1.57" />
-      <geometry>
-        <mesh filename="file://$(find quadruped_description)//meshes/joint_gear_upper_assembly.stl" />
-      </geometry>
-    </collision>
-  </link>
-  <link name="back_left_u">
-    <inertial>
-      <mass value="0.814" />
-      <inertia ixx="7701247.352E-09" ixy="96047.710E-09"  ixz="-1228944.675E-09"
-               iyy="7801785.041E-09" iyz="550113.749E-09"
-               izz="877983.793E-09" />
-    </inertial>
-    <visual>
-      <origin rpy="1.57 3.14 1.57" xyz="0 0 0"/>
-      <geometry>
-        <mesh filename="file://$(find quadruped_description)//meshes/joint_gear_upper_assembly.stl" />
-      </geometry>
-      <material name="grey"/>
-    </visual>
-    <collision>
-      <origin
-        xyz="0 0 0"
-        rpy="1.57 3.14 1.57" />
-      <geometry>
-        <mesh filename="file://$(find quadruped_description)//meshes/joint_gear_upper_assembly.stl" />
-      </geometry>
-    </collision>
-  </link>
-  <link name="back_right_u">
-    <inertial>
-      <mass value="0.814" />
-      <inertia ixx="7701247.352E-09" ixy="96047.710E-09"  ixz="-1228944.675E-09"
-               iyy="7801785.041E-09" iyz="550113.749E-09"
-               izz="877983.793E-09" />
-    </inertial>
-    <visual>
-      <origin rpy="1.57 0 1.57" xyz="0 0 0"/>
-      <geometry>
-        <mesh filename="file://$(find quadruped_description)//meshes/joint_gear_upper_assembly.stl" />
-      </geometry>
-      <material name="grey"/>
-    </visual>
-    <collision>
-      <origin
-        xyz="0 0 0"
-        rpy="1.57 0 1.57" />
-      <geometry>
-        <mesh filename="file://$(find quadruped_description)//meshes/joint_gear_upper_assembly.stl" />
-      </geometry>
-    </collision>
-  </link>
-  <link name="front_left_d">
-    <inertial>
-      <mass value="0.5" />
-      <inertia ixx="7141392.287E-09" ixy="-13.226E-09"  ixz="-913664.184E-09"
-               iyy="7895374.282E-09" iyz="-31.485E-09"
-               izz="830881.651E-09" />
-    </inertial>
-    <visual>
-      <origin rpy="1.57 0 1.57" xyz="0 0 0"/>
-      <geometry>
-        <mesh filename="file://$(find quadruped_description)//meshes/Assembly_lower_link_v2.stl" />
-      </geometry>
-      <material name="grey"/>
-    </visual>
-    <collision>
-      <origin
-        xyz="0 0 0"
-        rpy="1.57 0 1.57" />
-      <geometry>
-        <mesh filename="file://$(find quadruped_description)//meshes/Assembly_lower_link_v2.stl" />
-      </geometry>
-    </collision>
-  </link>
-  <link name="front_right_d">
-    <inertial>
-      <mass value="0.5" />
-      <inertia ixx="7141392.287E-09" ixy="-13.226E-09"  ixz="-913664.184E-09"
-               iyy="7895374.282E-09" iyz="-31.485E-09"
-               izz="830881.651E-09" />
-    </inertial>
-    <visual>
-      <origin rpy="-1.57 0 -1.57" xyz="0 0 0"/>
-      <geometry>
-        <mesh filename="file://$(find quadruped_description)//meshes/Assembly_lower_link_v2.stl" />
-      </geometry>
-      <material name="grey"/>
-    </visual>
-    <collision>
-      <origin
-        xyz="0 0 0"
-        rpy="-1.57 0 -1.57" />
-      <geometry>
-        <mesh filename="file://$(find quadruped_description)//meshes/Assembly_lower_link_v2.stl" />
-      </geometry>
-    </collision>
-  </link>
-  <link name="back_left_d">
-    <inertial>
-      <mass value="0.5" />
-      <inertia ixx="7141392.287E-09" ixy="-13.226E-09"  ixz="-913664.184E-09"
-               iyy="7895374.282E-09" iyz="-31.485E-09"
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