Commit message: .

File: quadruped_description/urdf/quadruped_gazebo.urdf.xacro (robot description, xacro)
@@ -14,4 +14,8 @@
   </gazebo>
   <gazebo reference="back_left_d">
+    <mu1>0.20</mu1>
+    <mu2>0.20</mu2>
+  </gazebo>
+  <gazebo reference="body">
     <mu1>0.20</mu1>
     <mu2>0.20</mu2>

File: quadruped_description/urdf/quadruped_robot.urdf.xacro (robot description, xacro)
@@ -6,5 +6,9 @@
     <inertial>
       <mass
-        value="1" />
+        value="5" />
+      <!-- <inertia
+        ixx="0.04" ixy="-0.000009" ixz="0.0045"
+        iyy="0.043" iyz="-0.000022"
+        izz="0.03" /> -->
       <inertia
         ixx="0.08" ixy="-0.0000173" ixz="0.00929"
@@ -65,4 +69,7 @@
     <inertial>
       <mass value="0.8" />
+      <!-- <inertia ixx="0.00025" ixy="0.0012"  ixz="0.0"
+               iyy="0.022" iyz="0.0"
+               izz="0.022" /> -->
       <inertia ixx="0.00051" ixy="0.0025"  ixz="0.0"
                iyy="0.044" iyz="0.0"
@@ -88,4 +95,7 @@
     <inertial>
       <mass value="0.8" />
+      <!-- <inertia ixx="0.00035" ixy="-0.0019"  ixz="0.0"
+               iyy="0.022" iyz="0.0"
+               izz="0.022" /> -->
       <inertia ixx="0.00076" ixy="-0.00385"  ixz="0.0"
                iyy="0.044" iyz="0.0"
@@ -111,4 +121,7 @@
     <inertial>
       <mass value="0.8" />
+      <!-- <inertia ixx="0.00035" ixy="-0.0019"  ixz="0.0"
+               iyy="0.022" iyz="0.0"
+               izz="0.022" /> -->
       <inertia ixx="0.00076" ixy="-0.00385"  ixz="0.0"
                iyy="0.044" iyz="0.0"
@@ -134,4 +147,7 @@
     <inertial>
       <mass value="0.8" />
+      <!-- <inertia ixx="0.00025" ixy="0.0012"  ixz="0.0"
+               iyy="0.022" iyz="0.0"
+               izz="0.022" /> -->
       <inertia ixx="0.00051" ixy="0.0025"  ixz="0.0"
                iyy="0.044" iyz="0.0"
@@ -160,4 +176,7 @@
                iyy="0.1412" iyz="0.0"
                izz="0.1447" /> Pata nueva-->
+      <!-- <inertia ixx="0.000045" ixy="0.0019"  ixz="0.0"
+               iyy="0.022" iyz="0.0"
+               izz="0.022" /> -->
       <inertia ixx="0.0009" ixy="0.0038"  ixz="0.0"
                iyy="0.044" iyz="0.0"
@@ -183,4 +202,7 @@
     <inertial>
       <mass value="1.0" />
+      <!-- <inertia ixx="0.000045" ixy="-0.0019"  ixz="0.0"
+               iyy="0.022" iyz="0.0"
+               izz="0.022" /> -->
       <inertia ixx="0.0009" ixy="-0.0038"  ixz="0.0"
                iyy="0.044" iyz="0.0"
@@ -206,4 +228,7 @@
     <inertial>
       <mass value="1.0" />
+      <!-- <inertia ixx="0.000045" ixy="-0.0019"  ixz="0.0"
+               iyy="0.022" iyz="0.0"
+               izz="0.022" /> -->
       <inertia ixx="0.0009" ixy="-0.0038"  ixz="0.0"
                iyy="0.044" iyz="0.0"
@@ -229,4 +254,7 @@
     <inertial>
       <mass value="1.0" />
+      <!-- <inertia ixx="0.000045" ixy="0.0019"  ixz="0.0"
+               iyy="0.022" iyz="0.0"
+               izz="0.022" /> -->
       <inertia ixx="0.0009" ixy="0.0038"  ixz="0.0"
                iyy="0.044" iyz="0.0"

Commit message: .

File: quadruped_description/urdf/quadruped_gazebo.urdf.xacro (robot description, xacro)
@@ -2,20 +2,90 @@
 <robot xmlns:xacro="http://www.ros.org/wiki/xacro">
   <gazebo reference="front_left_d">
+    <material>
+      <script>
+        <uri>file://media/materials/scripts/gazebo.material</uri>
+        <name>Gazebo/Grey</name>
+      </script>
+    </material>
     <mu1>0.20</mu1>
     <mu2>0.20</mu2>
   </gazebo>
   <gazebo reference="front_right_d">
+    <material>
+      <script>
+        <uri>file://media/materials/scripts/gazebo.material</uri>
+        <name>Gazebo/Grey</name>
+      </script>
+    </material>
     <mu1>0.20</mu1>
     <mu2>0.20</mu2>
   </gazebo>
   <gazebo reference="back_right_d">
+    <material>
+      <script>
+        <uri>file://media/materials/scripts/gazebo.material</uri>
+        <name>Gazebo/Grey</name>
+      </script>
+    </material>
     <mu1>0.20</mu1>
     <mu2>0.20</mu2>
   </gazebo>
   <gazebo reference="back_left_d">
+    <material>
+      <script>
+        <uri>file://media/materials/scripts/gazebo.material</uri>
+        <name>Gazebo/Grey</name>
+      </script>
+    </material>
     <mu1>0.20</mu1>
     <mu2>0.20</mu2>
   </gazebo>
   <gazebo reference="body">
+    <material>
+      <script>
+        <uri>file://media/materials/scripts/gazebo.material</uri>
+        <name>Gazebo/Grey</name>
+      </script>
+    </material>
+    <mu1>0.20</mu1>
+    <mu2>0.20</mu2>
+  </gazebo>
+  <gazebo reference="front_left_u">
+    <material>
+      <script>
+        <uri>file://media/materials/scripts/gazebo.material</uri>
+        <name>Gazebo/Grey</name>
+      </script>
+    </material>
+    <mu1>0.20</mu1>
+    <mu2>0.20</mu2>
+  </gazebo>
+  <gazebo reference="front_right_u">
+    <material>
+      <script>
+        <uri>file://media/materials/scripts/gazebo.material</uri>
+        <name>Gazebo/Grey</name>
+      </script>
+    </material>
+    <mu1>0.20</mu1>
+    <mu2>0.20</mu2>
+  </gazebo>
+  <gazebo reference="back_right_u">
+    <material>
+      <script>
+        <uri>file://media/materials/scripts/gazebo.material</uri>
+        <name>Gazebo/Grey</name>
+      </script>
+    </material>
+    <mu1>0.20</mu1>
+    <mu2>0.20</mu2>
+  </gazebo>
+  <gazebo reference="back_left_u">
+    <material>
+      <script>
+        <uri>file://media/materials/scripts/gazebo.material</uri>
+        <name>Gazebo/Grey</name>
+      </script>
+    </material>
     <mu1>0.20</mu1>
     <mu2>0.20</mu2>

File: quadruped_description/urdf/quadruped_robot.urdf.xacro (robot description, xacro)
@@ -361,5 +361,5 @@
       <inertia ixx="1e-5" ixy="0" ixz="0" iyy="1e-5" iyz="0" izz="1e-5" />
     </inertial>
-    <visual>
+    <!-- <visual>
       <origin xyz="0 0.05 0" rpy="${pi/2} 0 0" />
       <geometry>
@@ -369,5 +369,5 @@
         <color rgba="0.5 0.5 0.5 1" />
       </material>
-    </visual>
+    </visual> -->
     <collision>
       <origin xyz="0 0.05 0" rpy="${pi/2} 0 0" />
@@ -388,5 +388,5 @@
       <inertia ixx="1e-5" ixy="0" ixz="0" iyy="1e-5" iyz="0" izz="1e-5" />
     </inertial>
-    <visual>
+    <!-- <visual>
       <origin xyz="0 -0.05 0" rpy="${pi/2} 0 0" />
       <geometry>
@@ -396,5 +396,5 @@
         <color rgba="0.5 0.5 0.5 1" />
       </material>
-    </visual>
+    </visual> -->
     <collision>
       <origin xyz="0 -0.05 0" rpy="${pi/2} 0 0" />
@@ -415,5 +415,5 @@
       <inertia ixx="1e-5" ixy="0" ixz="0" iyy="1e-5" iyz="0" izz="1e-5" />
     </inertial>
-    <visual>
+    <!-- <visual>
       <origin xyz="0 0.05 0" rpy="${pi/2} 0 0" />
       <geometry>
@@ -423,5 +423,5 @@
         <color rgba="0.5 0.5 0.5 1" />
       </material>
-    </visual>
+    </visual> -->
     <collision>
       <origin xyz="0 0.05 0" rpy="${pi/2} 0 0" />
@@ -442,5 +442,5 @@
       <inertia ixx="1e-5" ixy="0" ixz="0" iyy="1e-5" iyz="0" izz="1e-5" />
     </inertial>
-    <visual>
+    <!-- <visual>
       <origin xyz="0 -0.05 0" rpy="${pi/2} 0 0" />
       <geometry>
@@ -450,5 +450,5 @@
         <color rgba="0.5 0.5 0.5 1" />
       </material>
-    </visual>
+    </visual> -->
     <collision>
       <origin xyz="0 -0.05 0" rpy="${pi/2} 0 0" />

Commit message: Cambios en la simulacion  de gazebo y el xacro

File: quadruped_description/urdf/quadruped_gazebo.urdf.xacro (robot description, xacro)
@@ -2,92 +2,50 @@
 <robot xmlns:xacro="http://www.ros.org/wiki/xacro">
   <gazebo reference="front_left_d">
-    <material>
-      <script>
-        <uri>file://media/materials/scripts/gazebo.material</uri>
-        <name>Gazebo/Grey</name>
-      </script>
-    </material>
     <mu1>0.20</mu1>
     <mu2>0.20</mu2>
+    <material>Gazebo/FlatBlack</material>
   </gazebo>
   <gazebo reference="front_right_d">
-    <material>
-      <script>
-        <uri>file://media/materials/scripts/gazebo.material</uri>
-        <name>Gazebo/Grey</name>
-      </script>
-    </material>
     <mu1>0.20</mu1>
     <mu2>0.20</mu2>
+    <material>Gazebo/DarkGrey</material>
   </gazebo>
   <gazebo reference="back_right_d">
-    <material>
-      <script>
-        <uri>file://media/materials/scripts/gazebo.material</uri>
-        <name>Gazebo/Grey</name>
-      </script>
-    </material>
     <mu1>0.20</mu1>
     <mu2>0.20</mu2>
+    <material>Gazebo/DarkGrey</material>
   </gazebo>
   <gazebo reference="back_left_d">
-    <material>
-      <script>
-        <uri>file://media/materials/scripts/gazebo.material</uri>
-        <name>Gazebo/Grey</name>
-      </script>
-    </material>
     <mu1>0.20</mu1>
     <mu2>0.20</mu2>
+    <material>Gazebo/DarkGrey</material>
   </gazebo>
   <gazebo reference="body">
-    <material>
-      <script>
-        <uri>file://media/materials/scripts/gazebo.material</uri>
-        <name>Gazebo/Grey</name>
-      </script>
-    </material>
     <mu1>0.20</mu1>
     <mu2>0.20</mu2>
+    <material>Gazebo/FlatBlack</material>
   </gazebo>
   <gazebo reference="front_left_u">
-    <material>
-      <script>
-        <uri>file://media/materials/scripts/gazebo.material</uri>
-        <name>Gazebo/Grey</name>
-      </script>
-    </material>
     <mu1>0.20</mu1>
     <mu2>0.20</mu2>
+    <material>Gazebo/FlatBlack</material>
   </gazebo>
   <gazebo reference="front_right_u">
-    <material>
-      <script>
-        <uri>file://media/materials/scripts/gazebo.material</uri>
-        <name>Gazebo/Grey</name>
-      </script>
-    </material>
     <mu1>0.20</mu1>
     <mu2>0.20</mu2>
+    <material>Gazebo/FlatBlack</material>
   </gazebo>
   <gazebo reference="back_right_u">
-    <material>
-      <script>
-        <uri>file://media/materials/scripts/gazebo.material</uri>
-        <name>Gazebo/Grey</name>
-      </script>
-    </material>
     <mu1>0.20</mu1>
     <mu2>0.20</mu2>
+    <material>Gazebo/FlatBlack</material>
   </gazebo>
   <gazebo reference="back_left_u">
-    <material>
-      <script>
-        <uri>file://media/materials/scripts/gazebo.material</uri>
-        <name>Gazebo/Grey</name>
-      </script>
-    </material>
     <mu1>0.20</mu1>
     <mu2>0.20</mu2>
+    <material>Gazebo/FlatBlack</material>
+  </gazebo>
+  <gazebo reference="camera_link">
+    <material>Gazebo/Grey</material>
   </gazebo>
   <gazebo reference="front_left_d_contact_link">
